Commit message: Adjusted orientation of gripper inside the simulation environment

File: franka_description/robots/common/franka_robot.xacro (robot description, xacro)
@@ -9,5 +9,5 @@
                       parent:='world'
                       xyz:='0 0 0'
-                      rpy:='0 0 0'
+                      rpy:='0 0 ${-pi/4}'
                       hand:='true'
                       ee_id:=none
@@ -24,5 +24,5 @@
       arm_id="${arm_id}"
       xyz="${xyz}"
-      rpy="${rpy}"
+      rpy='0 0 0'
       safety_distance="0.03"
       gazebo="${gazebo}"
@@ -85,5 +85,5 @@
         </xacro:if>
         <joint name="${parent}_joint" type="fixed">
-          <origin xyz="${xyz}" rpy="${rpy}" />
+          <origin xyz="${xyz}" rpy="0 0 0" />
           <parent link="${parent}" />
           <child  link="${arm_id}_link0" />
