Commit message: Removed mimicked joints from franka hand for pinocchio compatibility

File: franka_description/end_effectors/common/franka_hand.xacro (robot description, xacro)
@@ -100,20 +100,20 @@
       </xacro:if>
     </link>
-    <joint name="${arm_id}_finger_joint1" type="prismatic">
+    <joint name="${arm_id}_finger_joint1" type="fixed">
       <parent link="${arm_id}_hand" />
       <child link="${arm_id}_leftfinger" />
       <origin xyz="0 0 0.0584" rpy="0 0 0" />
-      <axis xyz="0 1 0" />
+      <!-- <axis xyz="0 1 0" />
       <limit effort="100" lower="0.0" upper="0.04" velocity="0.2" />
-      <dynamics damping="0.3" />
+      <dynamics damping="0.3" /> -->
     </joint>
-    <joint name="${arm_id}_finger_joint2" type="prismatic">
+    <joint name="${arm_id}_finger_joint2" type="fixed">
       <parent link="${arm_id}_hand" />
       <child link="${arm_id}_rightfinger" />
       <origin xyz="0 0 0.0584" rpy="0 0 0" />
-      <axis xyz="0 -1 0" />
-      <limit effort="100" lower="0.0" upper="0.04" velocity="0.2" />
-      <mimic joint="${arm_id}_finger_joint1" />
-      <dynamics damping="0.3" />
+      <!-- <axis xyz="0 -1 0" />
+      <limit effort="100" lower="0.0" upper="0.04" velocity="0.2" /> -->
+      <!-- <mimic joint="${arm_id}_finger_joint1" /> -->
+      <!-- <dynamics damping="0.3" /> -->
     </joint>
   </xacro:macro>
